File: board/board.kicad_pcb (KiCad board)
At the start: 2 copper layers, 21 x 13 mm, 1 part

Commit message: initial
Parts:
- added C1: 22uF, Capacitor_SMD:C_0805_2012Metric, F.Cu at (153.0, 97.4)
- added C2: 22uF, Capacitor_SMD:C_0805_2012Metric, F.Cu at (151.0, 97.4)
- added C3: 22uF, Capacitor_SMD:C_0805_2012Metric, F.Cu at (149.0, 97.4)
- added C4: 22uF, Capacitor_SMD:C_0805_2012Metric, F.Cu at (147.0, 97.4)
- added C5: 100nF, Capacitor_SMD:C_0603_1608Metric, F.Cu at (154.8, 97.2)
- added J1: 011_GPIO, on_edge:on_edge_2x05_host, F.Cu at (161.0, 96.5)
- added J2: 011_GPIO, on_edge:on_edge_2x05_device, F.Cu at (140.0, 96.5)
- added J3: Conn_01x02_Pin, Connector_PinHeader_2.54mm:PinHeader_1x02_P2.54mm_Vertical, F.Cu at (149.5, 101.1)
- added R1: 0.2R, Capacitor_SMD:C_0603_1608Metric, F.Cu at (155.2, 91.6)
- added U1: DRV8870DDA, Package_SO:Texas_HTSOP-8-1EP_3.9x4.9mm_P1.27mm_EP2.95x4.9mm_Mask2.4x3.1mm_ThermalVias, F.Cu at (150.2, 92.9)
- LOGO1: moved to B.Cu
- moved LOGO1 1.43 mm to (150.1, 97.6), turned to 180 degrees
Routing:
- net GND: track 0.00 -> 52.9 mm, vias 0 -> 2
- net /mc/VREF: track 0.00 -> 26.1 mm, vias 0 -> 2
- net Net-(J1-5V): track 0.00 -> 17.9 mm
- net /mc/V+: track 0.00 -> 14.7 mm, vias 0 -> 1
- net /mc/OUT2: track 0.00 -> 10.0 mm, vias 0 -> 2
- net /mc/IN2: track 0.00 -> 7.59 mm, vias 0 -> 2
- net /mc/OUT1: track 0.00 -> 5.98 mm
- net /mc/IN1: track 0.00 -> 5.38 mm
- net /mc/ISEN: track 0.00 -> 2.17 mm
Other:
- outline, holes or cut-outs redrawn
- board text added: "+"
- board text added: "-"
- board text added: "osf.011"
- board text added: "osf.b159.v1.0"
