File: board/board.kicad_sch (KiCad schematic)
At the start: 1 part

Commit message: initial
Parts:
- added J1: 011_GPIO, on_edge:on_edge_2x05_host, symbol put_on_edge:011_GPIO
- added J2: 011_GPIO, on_edge:on_edge_2x05_device, symbol put_on_edge:011_GPIO
- added J3: Conn_01x02_Pin, Connector_PinHeader_2.54mm:PinHeader_1x02_P2.54mm_Vertical, symbol Connector:Conn_01x02_Pin
- added R1: 0.2R, Capacitor_SMD:C_0603_1608Metric, symbol Device:R_Small
Connections:
- net GND: now also J1.1 (GND), J1.8 (GND), J2.1 (GND), J2.8 (GND), J3.1 (Pin_1), R1.2
- new net: J1.10 (5V), J2.10 (5V)
- new net mc/IN1: J2.2 (GPIO0)
- new net mc/IN2: J2.3 (GPIO1)
- new net mc/ISEN: R1.1
- new net mc/OUT1: J1.2 (GPIO0)
- new net mc/OUT2: J1.3 (GPIO1)
- new net mc/V+: J3.2 (Pin_2)
- new net mc/VREF: J1.9 (3.3V), J2.9 (3.3V)
- no-connect marks 0 -> 8
Other:
- sheet implementation renamed mc
- sheet mc: file implementation.kicad_sch -> mc.kicad_sch
- sheet mc ports: added IN1, IN2, ISEN, OUT1, OUT2, V+, VREF; removed none
- note removed: "Input connectors go here"
- note removed: "Output connectors go here"
